Commit message: Added rviz debugging launch file ddrive_rviz and rviz testing configuration madbot.rviz, Added gazebo modifications to urdf, and debugged ddrive.urdf.xacro, as well as change dimensions of madbot and added new dependancies on Cmakelist

File: diff_drive/urdf/ddrive.urdf.xacro (robot description, xacro)
@@ -2,8 +2,8 @@
 <robot name="madbot" xmlns:xacro="https://www.ros.org/wiki/xacro">
     <!-- Get properties from madbot_dim.yaml configuration -->
-    <xacro:property name="madbot_yaml_file" value="$(find ddrive)/config/madbot_dim.yaml"/>
+    <xacro:property name="madbot_yaml_file" value="$(find diff_drive)/config/madbot_dim.yaml"/>
     <xacro:property name="madbot_dims" value="${load_yaml(madbot_yaml_file)}"/>
     <!-- Properties from madbot_dim.yaml -->
-    <xacro:property name="ddrive_dict" value="${madbot_dims['drive']}"/>
+    <xacro:property name="ddrive_dict" value="${madbot_dims['ddrive']}"/>
     <xacro:property name="rect_prism_dict" value="${ddrive_dict['rect_prism']}"/>
     <xacro:property name="rect_length" value="${rect_prism_dict['x_len']}"/>
@@ -15,4 +15,6 @@
     <xacro:property name="caster_dict" value="${ddrive_dict['caster']}"/>
     <xacro:property name="caster_radius" value="${caster_dict['radius']}"/>
+    <!-- Import all Gazebo-customization elements, including Gazebo colors -->
+    <xacro:include filename="$(find diff_drive)/urdf/ddrive.gazebo"/>
     <!-- Links -->
     <link name="rect_box">
@@ -20,5 +22,5 @@
             <origin xyz="0 0 0" rpy="0 0 0"/>
             <geometry>
-                <box "${rect_length} ${rect_width} ${rect_height}"/>
+                <box size="${rect_length} ${rect_width} ${rect_height}"/>
             </geometry>
         </visual>
@@ -26,5 +28,5 @@
             <origin xyz="0 0 0" rpy="0 0 0"/>
             <geometry>
-                <box "${rect_length} ${rect_width} ${rect_height}"/>
+                <box size="${rect_length} ${rect_width} ${rect_height}"/>
             </geometry>
         </collision>
@@ -90,5 +92,5 @@
     <link name="left_wheel">
         <visual>
-            <origin xyz="0 0 0" rpy="{pi/2} 0 0"/>
+            <origin xyz="0 0 0" rpy="${pi/2} 0 0"/>
             <geometry>
                 <cylinder length="${wheel_length}" radius="${wheel_radius}"/>
@@ -96,5 +98,5 @@
         </visual>
         <collision>
-            <origin xyz="0 0 0" rpy="{pi/2} 0 0"/>
+            <origin xyz="0 0 0" rpy="${pi/2} 0 0"/>
             <geometry>
                 <cylinder length="${wheel_length}" radius="${wheel_radius}"/>
@@ -114,5 +116,5 @@
     <link name="right_wheel">
         <visual>
-            <origin xyz="0 0 0" rpy="{pi/2} 0 0"/>
+            <origin xyz="0 0 0" rpy="${pi/2} 0 0"/>
             <geometry>
                 <cylinder length="${wheel_length}" radius="${wheel_radius}"/>
@@ -120,5 +122,5 @@
         </visual>
         <collision>
-            <origin xyz="0 0 0" rpy="{pi/2} 0 0"/>
+            <origin xyz="0 0 0" rpy="${pi/2} 0 0"/>
             <geometry>
                 <cylinder length="${wheel_length}" radius="${wheel_radius}"/>
@@ -147,14 +149,14 @@
         <origin xyz="${(1.0/3.0)*rect_length} 0 ${-(1.0/2.0)*rect_height}"/>
     </joint>
-    <joint name="left_drive" type="continous">
+    <joint name="left_drive" type="continuous">
         <parent link="rect_box"/>
         <child link="left_wheel"/>
-        <origin xyz="${-(1.0/3.0)*rect_length} -(1.0/2.0)*rect_width 0"/>
+        <origin xyz="${-(1.0/3.0)*rect_length} ${-(1.0/2.0)*(rect_width + wheel_length)} 0"/>
         <axis xyz="0 1 0"/>
     </joint>
-    <joint name="right_drive" type="continous">
+    <joint name="right_drive" type="continuous">
         <parent link="rect_box"/>
-        <child link="left_wheel"/>
-        <origin xyz="${-(1.0/3.0)*rect_length} (1.0/2.0)*rect_width 0"/>
+        <child link="right_wheel"/>
+        <origin xyz="${-(1.0/3.0)*rect_length} ${(1.0/2.0)*(rect_width + wheel_length)} 0"/>
         <axis xyz="0 1 0"/>
     </joint>

Commit message: Robot does flipy-flip with flip node

File: diff_drive/urdf/ddrive.urdf.xacro (robot description, xacro)
@@ -105,5 +105,5 @@
         <inertial>
             <origin xyz="0 0 0" rpy="0 0 0"/>
-            <mass value=".5"/>
+            <mass value="10"/>
             <inertia ixx="${((1.0/12.0)*(.5)*(3.0*wheel_radius**2 + wheel_length))}"
                     ixy="0"
@@ -129,5 +129,5 @@
         <inertial>
             <origin xyz="0 0 0" rpy="0 0 0"/>
-            <mass value=".5"/>
+            <mass value="10"/>
             <inertia ixx="${((1.0/12.0)*(.5)*(3.0*wheel_radius**2 + wheel_length))}"
                     ixy="0"
